Commit message: sensors configured

File: urdf/nick_bot.xacro (robot description, xacro)
@@ -1,5 +1,5 @@
 <?xml version='1.0'?>
 <robot name="nick_bot" xmlns:xacro="http://www.ros.org/wiki/xacro">
-    <xacro:include filename="$(find slam_project)/urdf/nick_bot.gazebo" />
+    <xacro:include filename="$(find slam_project)/urdf/nick_bot.gazebo"/>
     <link name="robot_footprint"></link>
     <joint name="robot_footprint_joint" type="fixed">
@@ -83,9 +83,15 @@
         </visual>
     </link>
-    <joint type="fixed" name="camera_joint">
+    <joint type="fixed" name="camera_link">
         <origin xyz="0.25 0 0" rpy="0 0 0"/>
         <child link="camera"/>
         <parent link="chassis"/>
     </joint>
+    <joint name="camera_joint" type="fixed">
+        <origin xyz="0 0 0" rpy="-1.5707 0 -1.5707"/>
+        <parent link="camera"/>
+        <child link="camera_rgbd_frame"/>
+    </joint>
+    <link name="camera_rgbd_frame"/>
     <link name='hokuyo'>
         <inertial>

Commit message: fixing git

File: urdf/nick_bot.xacro (robot description, xacro)
@@ -84,5 +84,5 @@
     </link>
     <joint type="fixed" name="camera_link">
-        <origin xyz="0.25 0 0" rpy="0 0 0"/>
+        <origin xyz="0.25 0 0.05" rpy="0 0 0"/>
         <child link="camera"/>
         <parent link="chassis"/>
